File: tACS_precision/tACS_precision_revised.brd (EAGLE design)
At the start: 49.2 x 49.5 mm, 48 parts, among them IC1 TLC2252, IC2 LM4040, IC3 TLC2252, IC4 LM4040, IC5 ADR5041, IC6 REF5050AIDR, IC7 78L05ACD, T1 FMMT734, T2 FMMT634, T3 FMMT634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

Commit message: including revised board files
Parts:
- IC7: value 78L05ACD -> L78L05
- moved TP6 2.01 mm to (47.6, 46.4)
- moved TP8 2.01 mm to (47.6, 43.8)
- moved H2 1.42 mm to (6.99, 41.9)
- moved H1 0.90 mm to (43.8, 6.99)
- moved IC5 0.64 mm to (27.9, 43.8)
- moved LED1 0.64 mm to (16.5, 34.9)
- moved LED2 0.64 mm to (21.6, 34.9)
- moved R6 0.64 mm to (17.8, 43.8)
- moved R9 0.64 mm to (25.4, 32.4)
- moved T5 0.64 mm to (43.2, 32.4)
- moved IC6 0.64 mm to (30.5, 19.7)
- moved R10 0.64 mm to (22.9, 28.6)
- moved R3 0.64 mm to (41.9, 17.1)
- moved R4 0.64 mm to (39.4, 17.1)
- moved R7 0.64 mm to (16.5, 27.3)
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Routing:
- net N$3: track 119.8 -> 116.9 mm, vias 4 -> 6
- net N$11: track 69.3 -> 71.3 mm
- net N$24: track 13.6 -> 15.5 mm
Other:
- board size 49.2 x 49.5 mm -> 51.1 x 48.9 mm
- board text added: "ELECTRICAL ISOLATION"
- board text removed: "- ELECTRICAL ISOLATION -"

Commit message: patched board layout
Parts:
- removed IC5: ADR5041, texas:DBZ_R-PDSO-G3
- added U$3: ADR5041, precision_tACS:SC70-3
- moved H2 7.01 mm to (7.62, 48.9)
- moved T3 5.85 mm to (20.3, 34.3)
- moved H1 4.49 mm to (48.3, 7.62)
- moved R9 4.07 mm to (27.9, 35.6)
- moved R3 4.07 mm to (44.5, 20.3)
- moved IC6 4.07 mm to (33.0, 22.9)
- moved LED1 4.07 mm to (19.1, 38.1)
- moved LED2 4.07 mm to (24.1, 38.1)
- moved R13 4.07 mm to (40.6, 44.5)
- moved R6 4.07 mm to (20.3, 47.0)
- moved T5 4.07 mm to (45.7, 35.6)
- moved TP6 4.07 mm to (50.2, 49.5)
- moved TP8 4.07 mm to (50.2, 47.0)
- moved TP9 4.07 mm to (6.35, 37.5)
- moved R12 4.07 mm to (48.9, 21.0)
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Connections:
- net N$15: now also U$3.ANODE; no longer IC5.2
- net N$16: now also U$3.CATHODE; no longer IC5.1
Routing:
- net N$3: track 116.9 -> 121.7 mm, vias 6 -> 4
- net N$2: track 6.20 -> 4.35 mm
- net N$9: track 17.2 -> 16.3 mm
Other:
- board size 51.1 x 48.9 mm -> 56.2 x 56.5 mm
- board text added: "ISO/+36V"
- board text added: "ISO/-36V"
- board text added: "ISO/GND"
- board text removed: "ISO|+36V"
- board text removed: "ISO|-36V"
- board text removed: "ISO|GND"

Commit message: Board fixed, firmware written, all tested
Parts:
- moved R11 4.02 mm to (29.8, 46.4)
- moved U$3 2.84 mm to (31.8, 49.5)
Connections:
- net N$15: now also IC1.4, R11.1; no longer U$3.ANODE
- net N$16: now also R11.2, U$3.ANODE; no longer IC1.4, R11.1, U$3.CATHODE
- net N$8: now also U$3.CATHODE; no longer R11.2
Routing:
- net N$16: track 26.6 -> 22.8 mm
- net N$15: track 16.1 -> 17.3 mm
- net N$8: track 43.7 -> 44.7 mm
